File: photodiode_sensor_board.kicad_pcb (KiCad board)
At the start: 2 copper layers, 110 x 40 mm, 10 parts, among them J1 Conn_Coaxial, J2 Conn_Coaxial, J3 Conn_Coaxial

Commit message: Add files via upload
Parts:
- D1: value G12183-003K -> STO46P_TO-18_SOCKET; footprint Package_TO_SOT_THT:TO-18-3_Window -> my_components:STO46P_TO-18_SOCKET
- D2: value MTPD1346D-100 -> STO46P_TO-18_SOCKET; footprint Package_TO_SOT_THT:TO-46-3_Window -> my_components:STO46P_TO-18_SOCKET
- D3: value BPW21R -> STO5P_TO-5_SOCKET; footprint Package_TO_SOT_THT:TO-5-2_Window -> my_components:STO5P_TO-5_SOCKET
- moved D3 2.50 mm to (100.1, 100.0), turned to 90 degrees
- moved D2 1.33 mm to (170.5, 100.0), turned to 180 degrees
- moved D1 1.27 mm to (134.8, 99.7), turned to 90 degrees
- renumbered REF** to M3
Connections:
- D3 pad 1: GND -> Net-(D3-Pad1)
- D3 pad 2: Net-(D3-Pad2) -> GND
- J3 pad 1: Net-(D3-Pad2) -> Net-(D3-Pad1)
Routing:
- net Net-(D3-Pad1): track 0.00 -> 31.6 mm
- net Net-(D3-Pad2): track 28.0 -> 0.00 mm
- net Net-(D1-Pad1): track 7.58 -> 6.36 mm
- net GND: vias 84 -> 85
Other:
- board text added: "L-PBF optical monitoring sensor board Rev. 1 by Marcel Meyer Garcia @ wbk KIT"
- board text added: "SMA1"
- board text added: "SMA2"
- board text added: "SMA3"
- board text added: "Thorlabs FD05D"
- board text added: "Thorlabs FGA015"
- board text added: "Vishay BPW21 R"
