File: photodiode_sensor_board.sch (KiCad schematic (older format))
At the start: 6 parts, among them J1 Conn_Coaxial, J2 Conn_Coaxial, J3 Conn_Coaxial

Commit message: Add files via upload
Parts:
- removed D1: G12183-003K, Package_TO_SOT_THT:TO-18-3_Window, symbol g12183-003k:G12183-003K
- removed D2: MTPD1346D-100, Package_TO_SOT_THT:TO-46-3_Window, symbol mtpd1346d-100:MTPD1346D-100
- removed D3: BPW21R, Package_TO_SOT_THT:TO-5-2_Window, symbol bpw21r:BPW21R
- added D1, D2: STO46P_TO-18_SOCKET, my_components:STO46P_TO-18_SOCKET, symbol sto46p_to-18_socket:STO46P_TO-18_SOCKET
- added D3: STO5P_TO-5_SOCKET, my_components:STO5P_TO-5_SOCKET, symbol sto5p_to-5_socket:STO5P_TO-5_SOCKET
Connections:
- net GND: now also D1.2 (ANODE), D1.3 (CASE), D2.2 (ANODE), D2.3 (CASE), D3.2 (ANODE)
- net at J1.1 (In): now also D1.1 (KATHODE)
- net at J2.1 (In): now also D2.1 (KATHODE)
- net at J3.1 (In): now also D3.1 (KATHODE)
- no-connect marks 0 -> 1
Changed lines of the file:
@@
 EESchema Schematic File Version 4
+LIBS:photodiode_sensor_board-cache
 EELAYER 26 0
 EELAYER END
@@
 $EndComp
 Connection ~ 8700 3150
-$Comp
-L mtpd1346d-100:MTPD1346D-100 D2
-U 1 1 5DB8193F
-P 6850 3050
-F 0 "D2" V 6753 3209 50  0000 L CNN
-F 1 "MTPD1346D-100" V 6846 3209 50  0000 L CNN
-F 2 "Package_TO_SOT_THT:TO-46-3_Window" H 6850 3225 50  0001 C CNN
-F 3 "" H 6800 3050 50  0001 C CNN
-	1    6850 3050
-	0    -1   1    0
-$EndComp
 Wire Wire Line
 	6850 2850 7050 2850
@@
 	1    7100 3150
 	1    0    0    -1
-$EndComp
-$Comp
-L g12183-003k:G12183-003K D1
-U 1 1 5DB81EDE
-P 4950 3050
-F 0 "D1" V 4853 3209 50  0000 L CNN
-F 1 "G12183-003K" V 4946 3209 50  0000 L CNN
-F 2 "Package_TO_SOT_THT:TO-18-3_Window" H 4950 3225 50  0001 C CNN
-F 3 "http://www.farnell.com/datasheets/2822644.pdf" H 4900 3050 50  0001 C CNN
-	1    4950 3050
-	0    -1   1    0
 $EndComp
 Wire Wire Line
@@
 $EndComp
 $Comp
-L bpw21r:BPW21R D3
-U 1 1 5DB832B5
+L sto46p_to-18_socket:STO46P_TO-18_SOCKET D1
+U 1 1 5DCBFC4C
+P 4950 3050
+F 0 "D1" V 4853 3209 50  0000 L CNN
+F 1 "STO46P_TO-18_SOCKET" V 4946 3209 50  0000 L CNN
+F 2 "my_components:STO46P_TO-18_SOCKET" H 4950 3225 50  0001 C CNN
+F 3 "https://marktechopto.com/pdf/products/datasheet/MTPD1346D-100.pdf" H 4900 3050 50  0001 C CNN
+	1    4950 3050
+	0    -1   1    0
+$EndComp
+$Comp
+L sto46p_to-18_socket:STO46P_TO-18_SOCKET D2
+U 1 1 5DCBFE74
+P 6850 3050
+F 0 "D2" V 6753 3209 50  0000 L CNN
+F 1 "STO46P_TO-18_SOCKET" V 6846 3209 50  0000 L CNN
+F 2 "my_components:STO46P_TO-18_SOCKET" H 6850 3225 50  0001 C CNN
+F 3 "https://marktechopto.com/pdf/products/datasheet/MTPD1346D-100.pdf" H 6800 3050 50  0001 C CNN
+	1    6850 3050
+	0    -1   1    0
+$EndComp
+$Comp
+L sto5p_to-5_socket:STO5P_TO-5_SOCKET D3
+U 1 1 5DCC0001
 P 8150 3050
 F 0 "D3" V 8053 3209 50  0000 L CNN
-F 1 "BPW21R" V 8146 3209 50  0000 L CNN
-F 2 "Package_TO_SOT_THT:TO-5-2_Window" H 8150 3225 50  0001 C CNN
-F 3 "https://www.vishay.com/docs/81519/bpw21r.pdf" H 8100 3050 50  0001 C CNN
+F 1 "STO5P_TO-5_SOCKET" V 8146 3209 50  0000 L CNN
+F 2 "my_components:STO5P_TO-5_SOCKET" H 8150 3225 50  0001 C CNN
+F 3 "https://marktechopto.com/pdf/products/datasheet/MTPD1346D-100.pdf" H 8100 3050 50  0001 C CNN
 	1    8150 3050
-	0    1    1    0
+	0    -1   1    0
 $EndComp
+NoConn ~ 8300 3000
 $EndSCHEMATC
